File: Type-C_IO_Shield_For_UNO.kicad_pcb (KiCad board)
At the start: 2 copper layers, 68.6 x 53.3 mm, 44 parts, among them J1 Conn_01x04, J10 Conn_01x04, J11 Conn_01x04, J12 Conn_01x04, J13 Conn_01x04, J14 Conn_01x04, J15 Conn_01x04, J17 Conn_01x06, J18 Conn_01x06, J19 Conn_01x06, J2 Conn_01x04, J21 Conn_01x04, J22 Conn_01x04, J23 Conn_01x04, J24 Conn_01x04, J25 Conn_01x04, J26 Conn_01x06, J27 Conn_01x06, J28 Screw_Terminal_01x02, J3 Conn_01x04, J4 USB_C_Receptacle_USB2.0, J5 Conn_01x04, J6 Conn_01x04, J7 Conn_01x04, P1 Power, P2 Analog, P3 Digital, P4 Digital, P5 CONN_01X01, P6 CONN_01X01, P7 CONN_01X01, P8 CONN_01X01, SW1 SW_SPST, U1 CH340C

Commit message: V1.2
Routing:
- net /A3: track 58.5 -> 43.1 mm
- net /A2: track 50.0 -> 36.9 mm
- net /A4(SDA): track 49.6 -> 38.6 mm
- net /A5(SCL): track 55.0 -> 44.0 mm
- net /1(Tx): track 147.5 -> 138.3 mm
- net +5V: track 187.9 -> 185.4 mm

Commit message: update usb location
Signed-off-by: St.kai <St.kai@live.cn>
Parts:
- moved J4 1.02 mm to (115.7, 88.3)
Routing:
- net Net-(J4-PadA7): track 47.8 -> 46.4 mm
- net Net-(J4-PadA6): track 46.2 -> 45.4 mm
Changed lines of the file:
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@@
   )
   (footprint "Connector_USB:USB_C_Receptacle_Palconn_UTC16-G" (layer "F.Cu")
-    (at 116.699 88.265 -90)
+    (at 115.683 88.265 -90)
     (descr "http://www.palpilot.com/wp-content/uploads/2017/05/UTC027-GKN-OR-Rev-A.pdf")
     (tags "USB C Type-C Receptacle USB2.0")
@@
   (segment (start 170.767511 101.044511) (end 170.767511 105.965489) (width 0.6) (layer "B.Cu") (net 3))
   (segment (start 135.138 115.57) (end 140.843 115.57) (width 0.6) (layer "B.Cu") (net 3))
-  (segment (start 119.209 91.465) (end 119.489 91.465) (width 0.6) (layer "F.Cu") (net 4))
   (segment (start 125.452 119.253) (end 123.952 119.253) (width 0.6) (layer "F.Cu") (net 5))
   (segment (start 135.128 125.349) (end 131.548 125.349) (width 0.6) (layer "F.Cu") (net 5))
@@
   (segment (start 135.128 88.265) (end 133.858 89.535) (width 0.2) (layer "F.Cu") (net 28))
   (segment (start 133.858 89.535) (end 135.806551 91.483551) (width 0.2) (layer "F.Cu") (net 28))
-  (segment (start 119.209 85.865) (end 120.389 85.865) (width 0.6) (layer "F.Cu") (net 29))
-  (segment (start 120.389 85.865) (end 120.904 86.38) (width 0.6) (layer "F.Cu") (net 29))
-  (segment (start 125.3705 94.0015) (end 122.034 90.665) (width 0.6) (layer "F.Cu") (net 29))
-  (segment (start 125.3705 95.885) (end 125.3705 94.0015) (width 0.6) (layer "F.Cu") (net 29))
-  (segment (start 122.034 90.665) (end 119.209 90.665) (width 0.6) (layer "F.Cu") (net 29))
-  (segment (start 120.904 90.15) (end 120.389 90.665) (width 0.6) (layer "F.Cu") (net 29))
-  (segment (start 120.904 86.38) (end 120.904 90.15) (width 0.6) (layer "F.Cu") (net 29))
-  (segment (start 120.389 90.665) (end 119.209 90.665) (width 0.6) (layer "F.Cu") (net 29))
+  (segment (start 119.272022 90.665) (end 118.193 90.665) (width 0.6) (layer "F.Cu") (net 29))
+  (segment (start 118.193 90.665) (end 120.1505 90.665) (width 0.6) (layer "F.Cu") (net 29))
+  (segment (start 119.672031 86.164031) (end 119.672031 90.264991) (width 0.6) (layer "F.Cu") (net 29))
+  (segment (start 119.373 85.865) (end 119.672031 86.164031) (width 0.6) (layer "F.Cu") (net 29))
+  (segment (start 119.672031 90.264991) (end 119.272022 90.665) (width 0.6) (layer "F.Cu") (net 29))
+  (segment (start 120.1505 90.665) (end 125.3705 95.885) (width 0.6) (layer "F.Cu") (net 29))
+  (segment (start 118.193 85.865) (end 119.373 85.865) (width 0.6) (layer "F.Cu") (net 29))
+  (segment (start 112.941486 111.74148) (end 112.15952 110.959514) (width 0.2) (layer "F.Cu") (net 31))
+  (segment (start 123.825 105.41) (end 117.49352 111.74148) (width 0.2) (layer "F.Cu") (net 31))
+  (segment (start 119.072511 88.964511) (end 119.072511 88.065489) (width 0.2) (layer "F.Cu") (net 31))
+  (segment (start 119.022022 88.015) (end 118.193 88.015) (width 0.2) (layer "F.Cu") (net 31))
+  (segment (start 118.193 89.015) (end 119.022022 89.015) (width 0.2) (layer "F.Cu") (net 31))
+  (segment (start 118.193 89.015) (end 114.115006 89.015) (width 0.2) (layer "F.Cu") (net 31))
+  (segment (start 112.15952 90.970486) (end 114.115006 89.015) (width 0.2) (layer "F.Cu") (net 31))
+  (segment (start 112.15952 110.959514) (end 112.15952 90.970486) (width 0.2) (layer "F.Cu") (net 31))
+  (segment (start 119.072511 88.065489) (end 119.022022 88.015) (width 0.2) (layer "F.Cu") (net 31))
   (segment (start 117.49352 111.74148) (end 112.941486 111.74148) (width 0.2) (layer "F.Cu") (net 31))
-  (segment (start 115.494461 92.16048) (end 116.909194 92.16048) (width 0.2) (layer "F.Cu") (net 31))
-  (segment (start 119.209 89.015) (end 120.038022 89.015) (width 0.2) (layer "F.Cu") (net 31))
-  (segment (start 118.329489 89.065489) (end 119.209 89.065489) (width 0.2) (layer "F.Cu") (net 31))
-  (segment (start 116.909194 92.16048) (end 117.748979 91.320695) (width 0.2) (layer "F.Cu") (net 31))
-  (segment (start 120.088511 88.065489) (end 120.038022 88.015) (width 0.2) (layer "F.Cu") (net 31))
-  (segment (start 120.038022 88.015) (end 119.209 88.015) (width 0.2) (layer "F.Cu") (net 31))
-  (segment (start 123.825 105.41) (end 117.49352 111.74148) (width 0.2) (layer "F.Cu") (net 31))
-  (segment (start 113.748539 91.83548) (end 115.169461 91.83548) (width 0.2) (layer "F.Cu") (net 31))
-  (segment (start 119.209 89.065489) (end 119.209 89.015) (width 0.2) (layer "F.Cu") (net 31))
   (segment (start 125.033 105.41) (end 123.825 105.41) (width 0.2) (layer "F.Cu") (net 31))
-  (segment (start 115.169461 91.83548) (end 115.494461 92.16048) (width 0.2) (layer "F.Cu") (net 31))
-  (segment (start 117.748979 91.320695) (end 117.748979 89.645999) (width 0.2) (layer "F.Cu") (net 31))
-  (segment (start 120.038022 89.015) (end 120.088511 88.964511) (width 0.2) (layer "F.Cu") (net 31))
-  (segment (start 117.748979 89.645999) (end 118.329489 89.065489) (width 0.2) (layer "F.Cu") (net 31))
-  (segment (start 112.941486 111.74148) (end 112.15952 110.959514) (width 0.2) (layer "F.Cu") (net 31))
-  (segment (start 112.15952 110.959514) (end 112.15952 93.424499) (width 0.2) (layer "F.Cu") (net 31))
-  (segment (start 120.088511 88.964511) (end 120.088511 88.065489) (width 0.2) (layer "F.Cu") (net 31))
-  (segment (start 112.15952 93.424499) (end 113.748539 91.83548) (width 0.2) (layer "F.Cu") (net 31))
-  (segment (start 112.776 112.141) (end 111.76 111.125) (width 0.2) (layer "F.Cu") (net 32))
-  (segment (start 118.329489 87.565489) (end 118.329489 88.484489) (width 0.2) (layer "F.Cu") (net 32))
-  (segment (start 118.379978 87.515) (end 118.329489 87.565489) (width 0.2) (layer "F.Cu") (net 32))
-  (segment (start 115.05 87.515) (end 119.209 87.515) (width 0.2) (layer "F.Cu") (net 32))
-  (segment (start 123.120006 106.68) (end 117.659006 112.141) (width 0.2) (layer "F.Cu") (net 32))
-  (segment (start 125.033 106.68) (end 123.120006 106.68) (width 0.2) (layer "F.Cu") (net 32))
-  (segment (start 118.329489 88.484489) (end 118.36 88.515) (width 0.2) (layer "F.Cu") (net 32))
-  (segment (start 117.659006 112.141) (end 112.776 112.141) (width 0.2) (layer "F.Cu") (net 32))
-  (segment (start 111.76 90.805) (end 115.05 87.515) (width 0.2) (layer "F.Cu") (net 32))
-  (segment (start 111.76 111.125) (end 111.76 90.805) (width 0.2) (layer "F.Cu") (net 32))
-  (segment (start 118.36 88.515) (end 119.209 88.515) (width 0.2) (layer "F.Cu") (net 32))
-  (segment (start 119.209 87.515) (end 118.379978 87.515) (width 0.2) (layer "F.Cu") (net 32))
-  (segment (start 114.459 92.585) (end 118.629 92.585) (width 0.25) (layer "F.Cu") (net 36))
-  (segment (start 114.806 83.945) (end 114.808 83.947) (width 0.25) (layer "F.Cu") (net 36))
-  (segment (start 114.81 83.945) (end 118.629 83.945) (width 0.25) (layer "F.Cu") (net 36))
-  (segment (start 114.808 83.947) (end 114.81 83.945) (width 0.25) (layer "F.Cu") (net 36))
-  (segment (start 114.459 83.945) (end 114.806 83.945) (width 0.25) (layer "F.Cu") (net 36))
+  (segment (start 119.022022 89.015) (end 119.072511 88.964511) (width 0.2) (layer "F.Cu") (net 31))
+  (segment (start 114.05 88.515) (end 111.76 90.805) (width 0.2) (layer "F.Cu") (net 32))
+  (segment (start 117.363978 87.515) (end 118.193 87.515) (width 0.2) (layer "F.Cu") (net 32))
+  (segment (start 117.313489 88.464511) (end 117.313489 87.565489) (width 0.2) (layer "F.Cu") (net 32))
+  (segment (start 118.193 88.515) (end 117.363978 88.515) (width 0.2) (layer "F.Cu") (net 32))
+  (segment (start 123.120006 106.68) (end 125.033 106.68) (width 0.2) (layer "F.Cu") (net 32))
+  (segment (start 112.776 112.141) (end 117.659006 112.141) (width 0.2) (layer "F.Cu") (net 32))
+  (segment (start 111.76 90.805) (end 111.76 111.125) (width 0.2) (layer "F.Cu") (net 32))
+  (segment (start 117.363978 88.515) (end 117.313489 88.464511) (width 0.2) (layer "F.Cu") (net 32))
+  (segment (start 117.313489 87.565489) (end 117.363978 87.515) (width 0.2) (layer "F.Cu") (net 32))
+  (segment (start 118.193 88.515) (end 114.05 88.515) (width 0.2) (layer "F.Cu") (net 32))
+  (segment (start 111.76 111.125) (end 112.776 112.141) (width 0.2) (layer "F.Cu") (net 32))
+  (segment (start 117.659006 112.141) (end 123.120006 106.68) (width 0.2) (layer "F.Cu") (net 32))
+  (segment (start 113.443 92.585) (end 117.613 92.585) (width 0.2) (layer "F.Cu") (net 36))
+  (segment (start 113.443 83.945) (end 117.613 83.945) (width 0.2) (layer "F.Cu") (net 36))
   (segment (start 118.629 83.945) (end 118.629 92.585) (width 0.25) (layer "B.Cu") (net 36))
   (segment (start 161.798 99.695) (end 153.187031 91.084031) (width 0.2) (layer "F.Cu") (net 37))
@@
     (polygon
       (pts
-        (xy 175.514 73.533)
+        (xy 175.3616 73.279)
         (xy 176.784 74.803)
-        (xy 176.784 85.979)
+        (xy 176.784 86.233)
         (xy 179.324 88.773)
         (xy 179.324 92.329)
